Commit message: 好像没有很大问题，还在跑脚本

File: resources/robots/quad/quad.urdf (robot description, URDF)
Before this commit: robot quadrotor, 9 links, 8 joints
Links:
- link base_link: mass 0.225 -> 8.0

Commit message: 目前教师都不太收敛了，其他构建的差不多了

File: resources/robots/quad/quad.urdf (robot description, URDF)
Before this commit: robot quadrotor, 9 links, 8 joints
Links:
- link arm_motor_0: geometry visual cylinder length=0.225 radius=0.01
- link arm_motor_1: geometry visual cylinder length=0.225 radius=0.01
- link arm_motor_2: geometry visual cylinder length=0.225 radius=0.01
- link arm_motor_3: geometry visual cylinder length=0.225 radius=0.01
- link base_link: mass 0.225 -> 1.475; geometry collision sphere radius=0.25; visual sphere radius=0.08
- link motor_0: geometry visual cylinder length=0.05 radius=0.015
- link motor_1: geometry visual cylinder length=0.05 radius=0.015
- link motor_2: geometry visual cylinder length=0.05 radius=0.015
- link motor_3: geometry visual cylinder length=0.05 radius=0.015
Joints:
- joint base_link_to_arm_motor_0: origin xyz=0.065 -0.065 0.0 rpy=-1.5707963267948968 2.220446049250313e-16 -2.3561944901923453 -> xyz=0.0795 -0.0795 0.0 rpy=-1.5707963267948968 2.220446049250313e-16 -2.3561944901923453
- joint base_link_to_arm_motor_1: origin xyz=-0.065 -0.065 0.0 rpy=1.5707963267948968 2.220446049250313e-16 -0.7853981633974482 -> xyz=-0.0795 -0.0795 0.0 rpy=1.5707963267948968 2.220446049250313e-16 -0.7853981633974482
- joint base_link_to_arm_motor_2: origin xyz=-0.065 0.065 0.0 rpy=1.5707963267948968 0.0 -2.3561944901923453 -> xyz=-0.0795 0.0795 0.0 rpy=1.5707963267948968 0.0 -2.3561944901923453
- joint base_link_to_arm_motor_3: origin xyz=0.065 0.065 0.0 rpy=-1.5707963267948968 0.0 -0.7853981633974482 -> xyz=0.0795 0.0795 0.0 rpy=-1.5707963267948968 0.0 -0.7853981633974482
- joint base_link_to_motor_0: origin xyz=0.13 -0.13 0.0 rpy=0.0 0.0 0.0 -> xyz=0.159 -0.159 0.0 rpy=0.0 0.0 0.0
- joint base_link_to_motor_1: origin xyz=-0.13 -0.13 0.0 rpy=0.0 0.0 0.0 -> xyz=-0.159 -0.159 0.0 rpy=0.0 0.0 0.0
- joint base_link_to_motor_2: origin xyz=-0.13 0.13 0.0 rpy=0.0 0.0 0.0 -> xyz=-0.159 0.159 0.0 rpy=0.0 0.0 0.0
- joint base_link_to_motor_3: origin xyz=0.13 0.13 0.0 rpy=0.0 0.0 0.0 -> xyz=0.159 0.159 0.0 rpy=0.0 0.0 0.0
